File: noodle-spawnling-gecko.kicad_pcb (KiCad board)
At the start: 2 copper layers, 26 x 26 mm, 23 parts, among them J1 GPIO_PC1_PAD, J2 GPIO_PE13_PAD, J3 RESETn_PAD, J4 EXT_PWR_VDD, J5 EXT_PWR_GND, J6 LEU0/US0_HEADER, J7 DEBUG_HEADER, J8 USB_MICRO_B, SW1 CAP_TOUCH_BTN, U1 EFM32HG309

Commit message: add license to the silkscreen
Other:
- board text added: "CC-BY-SA 4.0"
Changed lines of the file:
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@@
     (area 36.924999 36.924999 63.075001 63.075001)
     (thickness 1.6)
-    (drawings 34)
+    (drawings 35)
     (tracks 293)
     (zones 0)
@@
     )
   )
+  (gr_text "CC-BY-SA 4.0" (at 50 58.4) (layer F.SilkS)
+    (effects (font (size 0.8 0.75) (thickness 0.15)))
+  )
   (gr_text 2 (at 57.5 55.8) (layer F.SilkS)
