File: noodle-spawnling-gecko.sch (KiCad schematic (older format))
At the start: 23 parts, among them J1 GPIO_PC1_PAD, J2 GPIO_PE13_PAD, J3 RESETn_PAD, J4 EXT_PWR_VDD, J5 EXT_PWR_GND, J6 LEU0/US0_HEADER, J7 DEBUG_HEADER, J8 USB_MICRO_B, SW1 CAP_TOUCH_BTN, U1 EFM32HG309

Commit message: add bom
Parts:
- BT1: MFR (none) -> Linx Technologies Inc.; MPN (none) -> BAT-HLD-001; SPN (none) -> BAT-HLD-001-ND; SPR (none) -> Digikey
- BZ1: MFR (none) -> Murata Electronics North America; MPN (none) -> PKMCS0909E4000-R1; SPN (none) -> 490-9647-1-ND; SPR (none) -> Digikey
- C1: MFR (none) -> Samsung Electro-Mechanics; MPN (none) -> CL05A475KQ5NRNC; SPN (none) -> 1276-1481-1-ND; SPR (none) -> Digikey
- C2, C3: MFR (none) -> Samsung Electro-Mechanics; MPN (none) -> CL05X105KQ5NNNC; SPN (none) -> 1276-1754-1-ND; SPR (none) -> Digikey
- C4: MFR (none) -> Murata Electronics North America; MPN (none) -> GRM155C80J106ME11D; SPN (none) -> 490-13233-1-ND; SPR (none) -> Digikey
- C5: MFR (none) -> Samsung Electro-Mechanics; MPN (none) -> CL05A104KQ5NNNC; SPN (none) -> 1276-1442-1-ND; SPR (none) -> Digikey
- D1, D2: MFR (none) -> Wurth Electronics Inc.; MPN (none) -> 151051SS04000; SPN (none) -> 732-11405-ND; SPR (none) -> Digikey
- J1, J2, J3, SW1: MFR (none) -> -; MPN (none) -> -; SPN (none) -> -; SPR (none) -> -
- J4, J5: MFR (none) -> Amphenol FCI; MPN (none) -> 68000-401HLF; SPN (none) -> 609-3466-ND; SPR (none) -> Digikey
- J6: MFR (none) -> Amphenol FCI; MPN (none) -> 20021121-00006C4LF; SPN (none) -> 609-3693-1-ND; SPR (none) -> Digikey
- J7: MFR (none) -> Sullins Connector Solutions; MPN (none) -> GRPB022VWQS-RC; SPN (none) -> S9012E-02-ND; SPR (none) -> Digikey
- J8: MFR (none) -> Molex, LLC; MPN (none) -> 1051330011; SPN (none) -> WM10134CT-ND; SPR (none) -> Digikey
- R1, R2: MFR (none) -> Yageo; MPN (none) -> RC0402FR-0752R3L; SPN (none) -> YAG3180CT-ND; SPR (none) -> Digikey
- R3, R4: MFR (none) -> Panasonic Electronic Components; MPN (none) -> ERJ-2RKF15R0X; SPN (none) -> P15.0LCT-ND; SPR (none) -> Digikey
- U1: MFR (none) -> Silicon Labs; MPN (none) -> EFM32HG309F64G-B-QFN24; SPN (none) -> 336-3896-ND; SPR (none) -> Digikey
